Commit message: fix: Replace hardcoded absolute paths with package:// URIs in URDF
- Replace all /home/raj/robo_ws hardcoded paths with package://pick_place_arm/
- Use package:// URI for mesh files (portable across systems)
- Use $(find) substitution for ros2_control.yaml parameter
- Makes project installable on any system without path modifications
- Critical fix for fresh installations on different machines

File: src/pick_place_arm/urdf/arm.urdf.xacro (robot description, xacro)
@@ -35,5 +35,5 @@
             <geometry>
                 <mesh
-                    filename="file:///home/raj/robo_ws/install/pick_place_arm/share/pick_place_arm/meshes/base_link.STL"
+                    filename="package://pick_place_arm/meshes/base_link.STL"
                     scale="1 1 1" />
             </geometry>
@@ -51,5 +51,5 @@
             <geometry>
                 <mesh
-                    filename="file:///home/raj/robo_ws/install/pick_place_arm/share/pick_place_arm/meshes/base_link.STL"
+                    filename="package://pick_place_arm/meshes/base_link.STL"
                     scale="1 1 1" />
             </geometry>
@@ -79,5 +79,5 @@
             <geometry>
                 <mesh
-                    filename="file:///home/raj/robo_ws/install/pick_place_arm/share/pick_place_arm/meshes/l1.STL"
+                    filename="package://pick_place_arm/meshes/l1.STL"
                     scale="1 1 1" />
             </geometry>
@@ -94,5 +94,5 @@
             <geometry>
                 <mesh
-                    filename="file:///home/raj/robo_ws/install/pick_place_arm/share/pick_place_arm/meshes/l1.STL"
+                    filename="package://pick_place_arm/meshes/l1.STL"
                     scale="1 1 1" />
             </geometry>
@@ -153,5 +153,5 @@
             <geometry>
                 <mesh
-                    filename="file:///home/raj/robo_ws/install/pick_place_arm/share/pick_place_arm/meshes/l2.STL"
+                    filename="package://pick_place_arm/meshes/l2.STL"
                     scale="1 1 1" />
             </geometry>
@@ -168,5 +168,5 @@
             <geometry>
                 <mesh
-                    filename="file:///home/raj/robo_ws/install/pick_place_arm/share/pick_place_arm/meshes/l2.STL"
+                    filename="package://pick_place_arm/meshes/l2.STL"
                     scale="1 1 1" />
             </geometry>
@@ -227,5 +227,5 @@
             <geometry>
                 <mesh
-                    filename="file:///home/raj/robo_ws/install/pick_place_arm/share/pick_place_arm/meshes/l3.STL"
+                    filename="package://pick_place_arm/meshes/l3.STL"
                     scale="1 1 1" />
             </geometry>
@@ -242,5 +242,5 @@
             <geometry>
                 <mesh
-                    filename="file:///home/raj/robo_ws/install/pick_place_arm/share/pick_place_arm/meshes/l3.STL"
+                    filename="package://pick_place_arm/meshes/l3.STL"
                     scale="1 1 1" />
             </geometry>
@@ -301,5 +301,5 @@
             <geometry>
                 <mesh
-                    filename="file:///home/raj/robo_ws/install/pick_place_arm/share/pick_place_arm/meshes/l4.STL"
+                    filename="package://pick_place_arm/meshes/l4.STL"
                     scale="1 1 1" />
             </geometry>
@@ -316,5 +316,5 @@
             <geometry>
                 <mesh
-                    filename="file:///home/raj/robo_ws/install/pick_place_arm/share/pick_place_arm/meshes/l4.STL"
+                    filename="package://pick_place_arm/meshes/l4.STL"
                     scale="1 1 1" />
             </geometry>
@@ -375,5 +375,5 @@
             <geometry>
                 <mesh
-                    filename="file:///home/raj/robo_ws/install/pick_place_arm/share/pick_place_arm/meshes/l5.STL"
+                    filename="package://pick_place_arm/meshes/l5.STL"
                     scale="1 1 1" />
             </geometry>
@@ -390,5 +390,5 @@
             <geometry>
                 <mesh
-                    filename="file:///home/raj/robo_ws/install/pick_place_arm/share/pick_place_arm/meshes/l5.STL"
+                    filename="package://pick_place_arm/meshes/l5.STL"
                     scale="1 1 1" />
             </geometry>
@@ -449,5 +449,5 @@
             <geometry>
                 <mesh
-                    filename="file:///home/raj/robo_ws/install/pick_place_arm/share/pick_place_arm/meshes/l6.STL"
+                    filename="package://pick_place_arm/meshes/l6.STL"
                     scale="1 1 1" />
             </geometry>
@@ -464,5 +464,5 @@
             <geometry>
                 <mesh
-                    filename="file:///home/raj/robo_ws/install/pick_place_arm/share/pick_place_arm/meshes/l6.STL"
+                    filename="package://pick_place_arm/meshes/l6.STL"
                     scale="1 1 1" />
             </geometry>
@@ -510,5 +510,5 @@
             <origin xyz="0 0 0" rpy="0 0 0" />
             <geometry>
-                <mesh filename="file:///home/raj/robo_ws/install/pick_place_arm/share/pick_place_arm/meshes/l7l.STL" scale="1 1 1" />
+                <mesh filename="package://pick_place_arm/meshes/l7l.STL" scale="1 1 1" />
             </geometry>
             <material name="">
@@ -519,5 +519,5 @@
             <origin xyz="0 0 0" rpy="0 0 0" />
             <geometry>
-                <mesh filename="file:///home/raj/robo_ws/install/pick_place_arm/share/pick_place_arm/meshes/l7l.STL" scale="1 1 1" />
+                <mesh filename="package://pick_place_arm/meshes/l7l.STL" scale="1 1 1" />
             </geometry>
         </collision>
@@ -558,5 +558,5 @@
             <origin xyz="0 0 0" rpy="0 0 0" />
             <geometry>
-                <mesh filename="file:///home/raj/robo_ws/install/pick_place_arm/share/pick_place_arm/meshes/l7r.STL" scale="1 1 1" />
+                <mesh filename="package://pick_place_arm/meshes/l7r.STL" scale="1 1 1" />
             </geometry>
             <material name="">
@@ -567,5 +567,5 @@
             <origin xyz="0 0 0" rpy="0 0 0" />
             <geometry>
-                <mesh filename="file:///home/raj/robo_ws/install/pick_place_arm/share/pick_place_arm/meshes/l7r.STL" scale="1 1 1" />
+                <mesh filename="package://pick_place_arm/meshes/l7r.STL" scale="1 1 1" />
             </geometry>
         </collision>
@@ -647,5 +647,5 @@
             <robot_param>robot_description</robot_param>
             <robot_param_node>robot_state_publisher</robot_param_node>
-            <parameters>/home/raj/robo_ws/install/pick_place_arm/share/pick_place_arm/config/ros2_control.yaml</parameters>
+            <parameters>$(find pick_place_arm)/config/ros2_control.yaml</parameters>
         </plugin>
     </gazebo>

Commit message: fix: Make URDF portable using xacro $(find) substitution
- Add mesh_path xacro property that uses $(find pick_place_arm)
- Replace all hardcoded /home/raj/robo_ws paths with ${mesh_path}
- Use $(find) for ros2_control.yaml parameter path
- Paths now resolve dynamically based on installation location
- Works on any system after colcon build

File: src/pick_place_arm/urdf/arm.urdf.xacro (robot description, xacro)
@@ -2,4 +2,6 @@
 <robot xmlns:xacro="http://www.ros.org/wiki/xacro" name="pick_place_arm">
     <xacro:arg name="gazebo_control" default="true" />
+    <xacro:arg name="mesh_path" default="file://$(find pick_place_arm)/meshes" />
+    <xacro:property name="mesh_path" value="$(arg mesh_path)" />
     <!-- Add dummy world link and fixed base_joint so base_link is not the URDF root
          (matches SRDF which declares base_joint and avoids KDL root-inertia warning) -->
@@ -35,5 +37,5 @@
             <geometry>
                 <mesh
-                    filename="package://pick_place_arm/meshes/base_link.STL"
+                    filename="${mesh_path}/base_link.STL"
                     scale="1 1 1" />
             </geometry>
@@ -51,5 +53,5 @@
             <geometry>
                 <mesh
-                    filename="package://pick_place_arm/meshes/base_link.STL"
+                    filename="${mesh_path}/base_link.STL"
                     scale="1 1 1" />
             </geometry>
@@ -79,5 +81,5 @@
             <geometry>
                 <mesh
-                    filename="package://pick_place_arm/meshes/l1.STL"
+                    filename="${mesh_path}/l1.STL"
                     scale="1 1 1" />
             </geometry>
@@ -94,5 +96,5 @@
             <geometry>
                 <mesh
-                    filename="package://pick_place_arm/meshes/l1.STL"
+                    filename="${mesh_path}/l1.STL"
                     scale="1 1 1" />
             </geometry>
@@ -153,5 +155,5 @@
             <geometry>
                 <mesh
-                    filename="package://pick_place_arm/meshes/l2.STL"
+                    filename="${mesh_path}/l2.STL"
                     scale="1 1 1" />
             </geometry>
@@ -168,5 +170,5 @@
             <geometry>
                 <mesh
-                    filename="package://pick_place_arm/meshes/l2.STL"
+                    filename="${mesh_path}/l2.STL"
                     scale="1 1 1" />
             </geometry>
@@ -227,5 +229,5 @@
             <geometry>
                 <mesh
-                    filename="package://pick_place_arm/meshes/l3.STL"
+                    filename="${mesh_path}/l3.STL"
                     scale="1 1 1" />
             </geometry>
@@ -242,5 +244,5 @@
             <geometry>
                 <mesh
-                    filename="package://pick_place_arm/meshes/l3.STL"
+                    filename="${mesh_path}/l3.STL"
                     scale="1 1 1" />
             </geometry>
@@ -301,5 +303,5 @@
             <geometry>
                 <mesh
-                    filename="package://pick_place_arm/meshes/l4.STL"
+                    filename="${mesh_path}/l4.STL"
                     scale="1 1 1" />
             </geometry>
@@ -316,5 +318,5 @@
             <geometry>
                 <mesh
-                    filename="package://pick_place_arm/meshes/l4.STL"
+                    filename="${mesh_path}/l4.STL"
                     scale="1 1 1" />
             </geometry>
@@ -375,5 +377,5 @@
             <geometry>
                 <mesh
-                    filename="package://pick_place_arm/meshes/l5.STL"
+                    filename="${mesh_path}/l5.STL"
                     scale="1 1 1" />
             </geometry>
@@ -390,5 +392,5 @@
             <geometry>
                 <mesh
-                    filename="package://pick_place_arm/meshes/l5.STL"
+                    filename="${mesh_path}/l5.STL"
                     scale="1 1 1" />
             </geometry>
@@ -449,5 +451,5 @@
             <geometry>
                 <mesh
-                    filename="package://pick_place_arm/meshes/l6.STL"
+                    filename="${mesh_path}/l6.STL"
                     scale="1 1 1" />
             </geometry>
@@ -464,5 +466,5 @@
             <geometry>
                 <mesh
-                    filename="package://pick_place_arm/meshes/l6.STL"
+                    filename="${mesh_path}/l6.STL"
                     scale="1 1 1" />
             </geometry>
@@ -510,5 +512,5 @@
             <origin xyz="0 0 0" rpy="0 0 0" />
             <geometry>
-                <mesh filename="package://pick_place_arm/meshes/l7l.STL" scale="1 1 1" />
+                <mesh filename="${mesh_path}/l7l.STL" scale="1 1 1" />
             </geometry>
             <material name="">
@@ -519,5 +521,5 @@
             <origin xyz="0 0 0" rpy="0 0 0" />
             <geometry>
-                <mesh filename="package://pick_place_arm/meshes/l7l.STL" scale="1 1 1" />
+                <mesh filename="${mesh_path}/l7l.STL" scale="1 1 1" />
             </geometry>
         </collision>
@@ -558,5 +560,5 @@
             <origin xyz="0 0 0" rpy="0 0 0" />
             <geometry>
-                <mesh filename="package://pick_place_arm/meshes/l7r.STL" scale="1 1 1" />
+                <mesh filename="${mesh_path}/l7r.STL" scale="1 1 1" />
             </geometry>
             <material name="">
@@ -567,5 +569,5 @@
             <origin xyz="0 0 0" rpy="0 0 0" />
             <geometry>
-                <mesh filename="package://pick_place_arm/meshes/l7r.STL" scale="1 1 1" />
+                <mesh filename="${mesh_path}/l7r.STL" scale="1 1 1" />
             </geometry>
         </collision>
